File: RelaisExpanderPrintV1.0/RelaisExpander Print V1.0/RelaisExpander Print V1.0.kicad_pcb (KiCad board)
At the start: 2 copper layers, 152 x 55 mm, 78 parts, among them J10 Screw_Terminal_01x03, J11 Screw_Terminal_01x03, J12 Screw_Terminal_01x03, J13 Screw_Terminal_01x03, J14 Screw_Terminal_01x03, J15 Screw_Terminal_01x03, J16 Screw_Terminal_01x03, J17 Screw_Terminal_01x03, J18 Screw_Terminal_01x03, J19 Screw_Terminal_01x03, J2 A0, J20 Screw_Terminal_01x03, J21 Screw_Terminal_01x03, J22 18-36V External Powersupply, J23 5V Out, J24 5V 3A Input, J25 I2C, J26 I2C, J3 A1, J5 A2, J6 Screw_Terminal_01x03, J7 Screw_Terminal_01x03, J8 Screw_Terminal_01x03, J9 Screw_Terminal_01x03, K1 G5LE-1, K10 G5LE-1, K11 G5LE-1, K12 G5LE-1, K13 G5LE-1, K14 G5LE-1, K15 G5LE-1, K16 G5LE-1, K2 G5LE-1, K3 G5LE-1, K4 G5LE-1, K5 G5LE-1, K6 G5LE-1, K7 G5LE-1, K8 G5LE-1, K9 G5LE-1, U1 AMS1117-3.3, U2 MCP23017_SP, U3 ULN2803A, U4 ULN2803A

Commit message: Minor Adjustments
Other:
- board text added: "I2C Address 0x20-0x27 0x20 = A0-A2 000: A0 = Bit 1 0x21 = A0-A2 001 A1 = Bit 2 0x22 = A0-A2 010 A2 = Bit 3 0x23 = A0-A2 011"
- board text added: "SCK"
- board text removed: "I2C Address 0x20-0x27 0x20 = A0-A2 000: A0 = Bit 1 0x21 = A0-A2 001 A1 = Bit 2 0x22 = A0-A2 010 A2 = Bit 3 0x23 = A0-A2 011 SCK SDA"
Changed lines of the file:
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@@
 		)
 		(property "Value" "3.3V"
-			(at 0 2.05 90)
-			(layer "F.Fab")
+			(at 0 3 180)
+			(layer "F.SilkS")
 			(effects
 				(font
@@
 		)
 		(property "Value" "SDA"
-			(at 0 2.05 0)
-			(layer "F.Fab")
+			(at -0.518177 2.334955 0)
+			(layer "F.SilkS")
 			(effects
 				(font
@@
 		(tags "Resistor Axial_DIN0207 series Axial Horizontal pin pitch 10.16mm 0.25W = 1/4W length 6.3mm diameter 2.5mm")
 		(property "Reference" "R16"
-			(at -2.42 0 0)
+			(at 0.185086 -1.664222 0)
 			(layer "F.SilkS")
 			(effects
@@
 		(property "Value" "5V"
 			(at 0 2.05 0)
-			(layer "F.Fab")
+			(layer "F.SilkS")
 			(effects
 				(font
@@
 		)
 		(property "Value" "SCK"
-			(at 0 2.05 0)
-			(layer "F.Fab")
+			(at 0.605933 2.380469 0)
+			(layer "F.SilkS")
 			(effects
 				(font
@@
 		(tags "THT Terminal Block Phoenix MPT-0,5-2-2.54 pitch 2.54mm size 5.54x6.2mm drill 1.1mm pad 2.2mm")
 		(property "Reference" "J26"
-			(at 1.27 -4.22 90)
+			(at 5.191923 1.758692 180)
 			(layer "F.SilkS")
 			(effects
@@
 		(tags "THT DIP DIL PDIP 2.54mm 7.62mm 300mil")
 		(property "Reference" "U4"
-			(at -1.88 4.54 180)
+			(at -1.685293 -1.131401 180)
 			(layer "F.SilkS")
 			(effects
@@
 		)
 		(property "Value" "5V"
-			(at 0 2.05 0)
-			(layer "F.Fab")
+			(at 0.261226 2.660894 0)
+			(layer "F.SilkS")
 			(effects
 				(font
@@
 		(tags "test point SMD pad")
 		(property "Reference" "TP5"
-			(at 0 -1.998 0)
+			(at -2.179907 -1.308077 0)
 			(layer "F.SilkS")
 			(effects
 				(font
-					(size 1 1)
+					(size 0.7 0.7)
 					(thickness 0.15)
 				)
@@
 		)
 		(property "Value" "External Supply"
-			(at 0 2.05 0)
-			(layer "F.Fab")
+			(at 1.729809 1.83189 0)
+			(layer "F.SilkS")
 			(effects
 				(font
-					(size 1 1)
+					(size 0.6 0.6)
 					(thickness 0.15)
 				)
@@
 		)
 		(fp_text user "${REFERENCE}"
-			(at 0 -2 0)
+			(at -2.576213 -1.38429 0)
 			(layer "F.Fab")
 			(effects
 				(font
-					(size 1 1)
+					(size 0.7 0.7)
 					(thickness 0.15)
 				)
@@
 		)
 		(property "Value" "5V 3A Input"
-			(at -7.73 1.8075 0)
+			(at -6.495914 1.785597 0)
 			(layer "F.SilkS")
 			(effects
@@
 		(layer "Edge.Cuts")
 	)
+	(gr_text "SCK"
+		(at 82.003548 84.370078 90)
+		(layer "F.SilkS")
+		(effects
+			(font
+				(size 0.7 0.7)
+				(thickness 0.175)
+				(bold yes)
+			)
+			(justify left bottom)
+		)
+	)
+	(gr_text "SCK"
+		(at 82.069396 89.242818 90)
+		(layer "F.SilkS")
+		(effects
+			(font
+				(size 0.7 0.7)
+				(thickness 0.175)
+				(bold yes)
+			)
+			(justify left bottom)
+		)
+	)
 	(gr_text "GND\nAX\n3.3V"
 		(at 171.5 89 0)
@@
 		)
 	)
-	(gr_text "I2C Address 0x20-0x27 \n0x20 = A0-A2 000:\nA0 = Bit 1 0x21 = A0-A2 001\nA1 = Bit 2 0x22 = A0-A2 010\nA2 = Bit 3 0x23 = A0-A2 011  SCK  	 SDA\n"
+	(gr_text "I2C Address 0x20-0x27 \n0x20 = A0-A2 000:\nA0 = Bit 1 0x21 = A0-A2 001\nA1 = Bit 2 0x22 = A0-A2 010\nA2 = Bit 3 0x23 = A0-A2 011\n"
 		(at 128 88 0)
 		(layer "F.SilkS")
@@
 	)
 	(gr_text "5V Power LED"
-		(at 182.5 81.5 0)
+		(at 181.82777 81.618526 0)
 		(layer "F.SilkS")
 		(effects
@@
 		)
 	)
-	(gr_text "+       -"
-		(at 172.5 83 0)
+	(gr_text "+  -"
+		(at 175.134406 83.626475 0)
 		(layer "F.SilkS")
 		(effects
@@
 	)
 	(via
-		(at 194.5 89)
+		(at 193.669501 88.665834)
 		(size 0.6)
 		(drill 0.3)

Commit message: Upload of Hauptprint
Routing:
- net Net-(U2-GPA2): track 51.0 -> 50.3 mm
- net +3.3V: track 152.1 -> 151.6 mm
- net GND: vias 144 -> 197
Other:
- board text added: "1 2 3"
- board text added: "Relais"
